Commit message: time trials setup and gui for drone control

File: drone_internals/urdf/quadcopter.xacro (robot description, xacro)
@@ -1,5 +1,5 @@
 <?xml version="1.0"?>
 <robot xmlns:xacro="http://wiki.ros.org/xacro" name="quadcopter">
-  <!-- properties -->
+  <!-- drone properties -->
   <xacro:property name="frame_radius" value="0.05"/>
   <xacro:property name="frame_height" value="0.025"/>
@@ -12,5 +12,10 @@
   <xacro:property name="propeller_height_offset" value="0.025"/>
   <xacro:property name="propeller_mass" value="0.01"/>
-   <xacro:macro name="cylinder_inertial" params="radius height mass *origin">
+  <!-- camera properties -->
+  <xacro:property name="camera_width" value="0.02"/>
+  <xacro:property name="camera_length" value="0.02"/>
+  <xacro:property name="camera_height" value="0.01"/>
+  <xacro:property name="camera_mass" value="0.01"/>
+  <xacro:macro name="cylinder_inertial" params="radius height mass *origin">
     <inertial>
       <mass value="${mass}"/>
@@ -24,4 +29,12 @@
         izz="${0.5 * mass * radius * radius}"
       />
+    </inertial>
+  </xacro:macro>
+  <xacro:macro name="box_inertial" params="name m x y z">
+    <inertial name="${name}_inertial">
+      <mass value="${m}"/>
+      <inertia  ixx="${m*(y*y+z*z)/12}" ixy = "0" ixz = "0"
+        iyy="${m*(x*x+y*y)/12}" iyz = "0"
+        izz="${m*(x*x+z*z)/12}"/>
     </inertial>
   </xacro:macro>
@@ -118,4 +131,5 @@
     <material>Gazebo/Orange</material>
   </gazebo>
+  <!-- defining 4 arms and propellors -->
   <xacro:arm i="1"/>
   <xacro:arm i="2"/>
@@ -126,4 +140,122 @@
   <xacro:propeller i="3" mat="Gazebo/BlueTransparent"/>
   <xacro:propeller i="4" mat="Gazebo/BlueTransparent"/>
+  <!-- cameras -->
+  <link name='camera1_link'>
+    <xacro:box_inertial name="camera1_link" m="${camera_mass}" x="${camera_width}" y="${camera_length}" z="${camera_height}"/>
+    <collision name='camera1_link_collision'>
+      <geometry>
+        <box size="${camera_length} ${camera_width} ${camera_height}"/>
+      </geometry>
+    </collision>
+    <visual name='camera1_link_visual'>
+      <origin xyz="0 0 0" rpy=" 0 0 0"/>
+      <geometry>
+        <box size="${camera_length} ${camera_width} ${camera_height}"/>
+      </geometry>
+    </visual>
+  </link>
+  <joint name="camera1_joint" type="fixed">
+    <parent link="frame"/>
+    <child link="camera1_link"/>
+    <origin xyz="${frame_radius} 0 0"/>
+  </joint>
+  <link name='camera2_link'>
+    <xacro:box_inertial name="camera2_link" m="${camera_mass}" x="${camera_width}" y="${camera_length}" z="${camera_height}"/>
+    <collision name='camera2_link_collision'>
+      <geometry>
+        <box size="${camera_length} ${camera_width} ${camera_height}"/>
+      </geometry>
+    </collision>
+    <visual name='camera2_link_visual'>
+      <origin xyz="0 0 0" rpy=" 0 0 0"/>
+      <geometry>
+        <box size="${camera_length} ${camera_width} ${camera_height}"/>
+      </geometry>
+    </visual>
+  </link>
+  <joint name="camera2_joint" type="fixed">
+    <parent link="frame"/>
+    <child link="camera2_link"/>
+    <origin xyz="0 0 ${frame_height/2}" rpy="0 -1.570796327 0"/>
+  </joint>
+  <!-- camera plugin -->
+  <gazebo reference="camera1_link">
+    <sensor type="camera" name="camera1">
+      <update_rate>30.0</update_rate>
+      <camera name="head">
+        <horizontal_fov>1.3962634</horizontal_fov>
+        <image>
+          <width>800</width>
+          <height>400</height>
+          <format>R8G8B8</format>
+        </image>
+        <clip>
+          <near>0.02</near>
+          <far>300</far>
+        </clip>
+        <noise>
+          <type>gaussian</type>
+          <!-- Noise is sampled independently per pixel on each frame.
+              That pixel's noise value is added to each of its color
+              channels, which at that point lie in the range [0,1]. -->
+          <mean>0.0</mean>
+          <stddev>0.007</stddev>
+        </noise>
+      </camera>
+      <plugin name="camera_controller" filename="libgazebo_ros_camera.so">
+        <alwaysOn>true</alwaysOn>
+        <updateRate>0.0</updateRate>
+        <cameraName>camera1</cameraName>
+        <imageTopicName>image_raw</imageTopicName>
+        <cameraInfoTopicName>camera_info</cameraInfoTopicName>
+        <frameName>camera1_link</frameName>
+        <hackBaseline>0.07</hackBaseline>
+        <distortionK1>0.0</distortionK1>
+        <distortionK2>0.0</distortionK2>
+        <distortionK3>0.0</distortionK3>
+        <distortionT1>0.0</distortionT1>
+        <distortionT2>0.0</distortionT2>
+      </plugin>
+    </sensor>
+  </gazebo>
+  <gazebo reference="camera2_link">
+    <sensor type="camera" name="camera2">
+      <update_rate>30.0</update_rate>
+      <camera name="head">
+        <horizontal_fov>1.3962634</horizontal_fov>
+        <image>
+          <width>64</width>
+          <height>64</height>
+          <format>R8G8B8</format>
+        </image>
+        <clip>
+          <near>0.02</near>
+          <far>300</far>
+        </clip>
+        <noise>
+          <type>gaussian</type>
+          <!-- Noise is sampled independently per pixel on each frame.
+              That pixel's noise value is added to each of its color
+              channels, which at that point lie in the range [0,1]. -->
+          <mean>0.0</mean>
+          <stddev>0.007</stddev>
+        </noise>
+      </camera>
+      <plugin name="camera_controller" filename="libgazebo_ros_camera.so">
+        <alwaysOn>true</alwaysOn>
+        <updateRate>0.0</updateRate>
+        <cameraName>camera2</cameraName>
+        <imageTopicName>image_raw</imageTopicName>
+        <cameraInfoTopicName>camera_info</cameraInfoTopicName>
+        <frameName>camera2_link</frameName>
+        <hackBaseline>0.07</hackBaseline>
+        <distortionK1>0.0</distortionK1>
+        <distortionK2>0.0</distortionK2>
+        <distortionK3>0.0</distortionK3>
+        <distortionT1>0.0</distortionT1>
+        <distortionT2>0.0</distortionT2>
+      </plugin>
+    </sensor>
+  </gazebo>
   <!-- motor control plugin-->
   <gazebo>

Commit message: Added line detection for the walls and improved the pitch detection

File: drone_internals/urdf/quadcopter.xacro (robot description, xacro)
@@ -17,4 +17,5 @@
   <xacro:property name="camera_height" value="0.01"/>
   <xacro:property name="camera_mass" value="0.01"/>
+  <xacro:property name="camera_fov" value="90"/>
   <xacro:macro name="cylinder_inertial" params="radius height mass *origin">
     <inertial>
@@ -177,5 +178,5 @@
     <parent link="frame"/>
     <child link="camera2_link"/>
-    <origin xyz="0 0 ${frame_height/2}" rpy="0 -1.570796327 0"/>
+    <origin xyz="0 0 ${frame_height/2}" rpy="0 -1.8 0"/>
   </joint>
   <!-- camera plugin -->
@@ -184,5 +185,5 @@
       <update_rate>30.0</update_rate>
       <camera name="head">
-        <horizontal_fov>1.3962634</horizontal_fov>
+        <horizontal_fov>1.57079632679</horizontal_fov>
         <image>
           <width>800</width>
@@ -223,8 +224,8 @@
       <update_rate>30.0</update_rate>
       <camera name="head">
-        <horizontal_fov>1.3962634</horizontal_fov>
+        <horizontal_fov>0.78539816339</horizontal_fov>
         <image>
-          <width>64</width>
-          <height>64</height>
+          <width>128</width>
+          <height>128</height>
           <format>R8G8B8</format>
         </image>

Commit message: got positioning working and lots of code cleanup

File: drone_internals/urdf/quadcopter.xacro (robot description, xacro)
@@ -139,7 +139,45 @@
   <xacro:propeller i="1" mat="Gazebo/RedTransparent"/>
   <xacro:propeller i="2" mat="Gazebo/RedTransparent"/>
-  <xacro:propeller i="3" mat="Gazebo/BlueTransparent"/>
-  <xacro:propeller i="4" mat="Gazebo/BlueTransparent"/>
+  <xacro:propeller i="3" mat="Gazebo/GreenTransparent"/>
+  <xacro:propeller i="4" mat="Gazebo/GreenTransparent"/>
   <!-- cameras -->
+  <link name='camera0_link'>
+    <xacro:box_inertial name="camera0_link" m="${camera_mass}" x="${camera_width}" y="${camera_length}" z="${camera_height}"/>
+    <collision name='camera0_link_collision'>
+      <geometry>
+        <box size="${camera_length} ${camera_width} ${camera_height}"/>
+      </geometry>
+    </collision>
+    <visual name='camera0_link_visual'>
+      <origin xyz="0 0 0" rpy=" 0 0 0"/>
+      <geometry>
+        <box size="${camera_length} ${camera_width} ${camera_height}"/>
+      </geometry>
+    </visual>
+  </link>
+  <joint name="camera0_joint" type="fixed">
+    <parent link="frame"/>
+    <child link="camera0_link"/>
+    <origin xyz="${frame_radius} 0 0"/>
+  </joint>
+  <link name='camera_top_link'>
+    <xacro:box_inertial name="camera_top_link" m="${camera_mass}" x="${camera_width}" y="${camera_length}" z="${camera_height}"/>
+    <collision name='camera_top_link_collision'>
+      <geometry>
+        <box size="${camera_length} ${camera_width} ${camera_height}"/>
+      </geometry>
+    </collision>
+    <visual name='camera_top_link_visual'>
+      <origin xyz="0 0 0" rpy=" 0 0 0"/>
+      <geometry>
+        <box size="${camera_length} ${camera_width} ${camera_height}"/>
+      </geometry>
+    </visual>
+  </link>
+  <joint name="camera_top_joint" type="fixed">
+    <parent link="frame"/>
+    <child link="camera_top_link"/>
+    <origin xyz="0 0 ${frame_height/2}" rpy="0 -1.8 0"/>
+  </joint>
   <link name='camera1_link'>
     <xacro:box_inertial name="camera1_link" m="${camera_mass}" x="${camera_width}" y="${camera_length}" z="${camera_height}"/>
@@ -159,26 +197,85 @@
     <parent link="frame"/>
     <child link="camera1_link"/>
-    <origin xyz="${frame_radius} 0 0"/>
-  </joint>
-  <link name='camera2_link'>
-    <xacro:box_inertial name="camera2_link" m="${camera_mass}" x="${camera_width}" y="${camera_length}" z="${camera_height}"/>
-    <collision name='camera2_link_collision'>
-      <geometry>
-        <box size="${camera_length} ${camera_width} ${camera_height}"/>
-      </geometry>
-    </collision>
-    <visual name='camera2_link_visual'>
-      <origin xyz="0 0 0" rpy=" 0 0 0"/>
-      <geometry>
-        <box size="${camera_length} ${camera_width} ${camera_height}"/>
-      </geometry>
-    </visual>
-  </link>
-  <joint name="camera2_joint" type="fixed">
-    <parent link="frame"/>
-    <child link="camera2_link"/>
-    <origin xyz="0 0 ${frame_height/2}" rpy="0 -1.8 0"/>
+    <origin xyz="${-1*frame_radius} 0 0" rpy="0 0 ${pi}"/>
   </joint>
   <!-- camera plugin -->
+  <gazebo reference="camera0_link">
+    <sensor type="camera" name="camera0">
+      <update_rate>30.0</update_rate>
+      <camera name="head">
+        <horizontal_fov>1.57079632679</horizontal_fov>
+        <image>
+          <width>800</width>
+          <height>400</height>
+          <format>R8G8B8</format>
+        </image>
+        <clip>
+          <near>0.02</near>
+          <far>300</far>
+        </clip>
+        <noise>
+          <type>gaussian</type>
+          <!-- Noise is sampled independently per pixel on each frame.
+              That pixel's noise value is added to each of its color
+              channels, which at that point lie in the range [0,1]. -->
+          <mean>0.0</mean>
+          <stddev>0.007</stddev>
+        </noise>
+      </camera>
+      <plugin name="camera_controller" filename="libgazebo_ros_camera.so">
+        <alwaysOn>true</alwaysOn>
+        <updateRate>0.0</updateRate>
+        <cameraName>camera0</cameraName>
+        <imageTopicName>image_raw</imageTopicName>
+        <cameraInfoTopicName>camera_info</cameraInfoTopicName>
+        <frameName>camera0_link</frameName>
+        <hackBaseline>0.07</hackBaseline>
+        <distortionK1>0.0</distortionK1>
+        <distortionK2>0.0</distortionK2>
+        <distortionK3>0.0</distortionK3>
+        <distortionT1>0.0</distortionT1>
+        <distortionT2>0.0</distortionT2>
+      </plugin>
+    </sensor>
+  </gazebo>
+  <gazebo reference="camera_top_link">
+    <sensor type="camera" name="camera_top">
+      <update_rate>30.0</update_rate>
+      <camera name="head">
+        <horizontal_fov>0.78539816339</horizontal_fov>
+        <image>
+          <width>128</width>
+          <height>128</height>
+          <format>R8G8B8</format>
+        </image>
+        <clip>
+          <near>0.02</near>
+          <far>300</far>
+        </clip>
+        <noise>
+          <type>gaussian</type>
+          <!-- Noise is sampled independently per pixel on each frame.
+              That pixel's noise value is added to each of its color
+              channels, which at that point lie in the range [0,1]. -->
+          <mean>0.0</mean>
+          <stddev>0.007</stddev>
+        </noise>
+      </camera>
+      <plugin name="camera_controller" filename="libgazebo_ros_camera.so">
+        <alwaysOn>true</alwaysOn>
+        <updateRate>0.0</updateRate>
+        <cameraName>camera_top</cameraName>
+        <imageTopicName>image_raw</imageTopicName>
+        <cameraInfoTopicName>camera_info</cameraInfoTopicName>
+        <frameName>camera_top_link</frameName>
+        <hackBaseline>0.07</hackBaseline>
+        <distortionK1>0.0</distortionK1>
+        <distortionK2>0.0</distortionK2>
+        <distortionK3>0.0</distortionK3>
+        <distortionT1>0.0</distortionT1>
+        <distortionT2>0.0</distortionT2>
+      </plugin>
+    </sensor>
+  </gazebo>
   <gazebo reference="camera1_link">
     <sensor type="camera" name="camera1">
@@ -220,43 +317,4 @@
     </sensor>
   </gazebo>
-  <gazebo reference="camera2_link">
-    <sensor type="camera" name="camera2">
-      <update_rate>30.0</update_rate>
-      <camera name="head">
-        <horizontal_fov>0.78539816339</horizontal_fov>
-        <image>
-          <width>128</width>
-          <height>128</height>
-          <format>R8G8B8</format>
-        </image>
-        <clip>
-          <near>0.02</near>
-          <far>300</far>
-        </clip>
-        <noise>
-          <type>gaussian</type>
-          <!-- Noise is sampled independently per pixel on each frame.
-              That pixel's noise value is added to each of its color
-              channels, which at that point lie in the range [0,1]. -->
-          <mean>0.0</mean>
-          <stddev>0.007</stddev>
-        </noise>
-      </camera>
-      <plugin name="camera_controller" filename="libgazebo_ros_camera.so">
-        <alwaysOn>true</alwaysOn>
-        <updateRate>0.0</updateRate>
-        <cameraName>camera2</cameraName>
-        <imageTopicName>image_raw</imageTopicName>
-        <cameraInfoTopicName>camera_info</cameraInfoTopicName>
-        <frameName>camera2_link</frameName>
-        <hackBaseline>0.07</hackBaseline>
-        <distortionK1>0.0</distortionK1>
-        <distortionK2>0.0</distortionK2>
-        <distortionK3>0.0</distortionK3>
-        <distortionT1>0.0</distortionT1>
-        <distortionT2>0.0</distortionT2>
-      </plugin>
-    </sensor>
-  </gazebo>
   <!-- motor control plugin-->
   <gazebo>
